File: iot-wifi-uno-hw.sch (KiCad schematic (older format))
At the start: 62 parts, among them CON1 BARREL_JACK, P1 CONN_01X08, P2 CONN_01X08, P3 CONN_01X06, P4 CONN_01X10, P5 CONN_01X04, Q1 Q_NPN_CBE, Q2 Q_NPN_CBE, U1 usb_mini_b, U2 BD00GA5WEFJ, U3 MCP16311-MNY, U4 CH340G, U5 ESP-12E, U6 MCP6001R, U7 MOSFET-P, X1 CRYSTAL_ABM3C

Commit message: Fix crystall of CH340G
Parts:
- C4, C5: value 8pF -> 22pF
Changed lines of the file:
@@
 P 1000 4950
 F 0 "C4" H 1092 4996 50  0000 L CNN
-F 1 "8pF" H 1092 4905 50  0000 L CNN
+F 1 "22pF" H 1092 4905 50  0000 L CNN
 F 2 "ESP8266:C_0603" H 1000 4950 50  0001 C CNN
 F 3 "" H 1000 4950 50  0000 C CNN
@@
 P 1850 4750
 F 0 "C5" H 1942 4796 50  0000 L CNN
-F 1 "8pF" H 1942 4705 50  0000 L CNN
+F 1 "22pF" H 1942 4705 50  0000 L CNN
 F 2 "ESP8266:C_0603" H 1850 4750 50  0001 C CNN
 F 3 "" H 1850 4750 50  0000 C CNN

Commit message: Modify footprint MCP16311, add zener to ADC, fix footprint 2 transistor
Parts:
- removed C7: 10uF/25v, ESP8266:C_0603, symbol C_Small
- removed C9: 10uF, ESP8266:C_0603, symbol C_Small
- removed D4: D, ESP8266:do214aa, symbol D
- added D1: SS24, ESP8266:do214aa, symbol D_Schottky_Small
- added D5: ZENER_3.3V, ESP8266:SOD-80, symbol ZENER_Small
- C15: renamed from C3; footprint Capacitors_SMD:C_1210_HandSoldering -> ESP8266:C_0603
- D3: renamed from D2; value ss24 -> SS24
- Q1, Q2: value Q_NPN_CBE -> MMBT8050LT1G; footprint TO_SOT_Packages_SMD:SOT-323 -> TO_SOT_Packages_SMD:SOT-23
- R10: renamed from R13; value 12K -> 10K
- R11: renamed from R14; value 12K -> 10K
- U7: value MOSFET-P -> IRLM6402
- renumbered C4 to C1, C15 to C10, C16 to C11, C10 to C12, C1 to C13, C17 to C14, C5 to C2, C11 to C3, C12 to C4, C2 to C5, C13 to C7, C14 to C9, D3 to D2, D1 to D4, GPIO0 to GPIO1, R11 to R12, R12 to R13, R17 to R14, R6 to R15, R7 to R16, R18 to R17, R21 to R18, R22 to R19, R19 to R20, R20 to R21, R8 to R22, R9 to R6, R10 to R7, R15 to R8, R16 to R9, U3 to U2, U4 to U3, U5 to U4, U6 to U5, U2 to U6
Connections:
- wire segments 230 -> 226
