File: iot-wifi-uno-hw.kicad_pcb (KiCad board)
At the start: 2 copper layers, 68.6 x 53.3 mm, 71 parts, among them CON1 BARREL_JACK, P1 CONN_01X08, P2 CONN_01X08, P3 CONN_01X06, P4 CONN_01X10, P5 CONN_01X04, Q1 Q_NPN_BEC, Q2 Q_NPN_BEC, SW1 RST, SW2 GPIO0, U1 usb_mini_b, U2 MCP16311-MNY, U3 CH340G, U4 ESP-12E, U5 MCP6001R, U6 BD00GA5WEFJ, U7 IRLM6402, X1 CRYSTAL_ABM3C

Commit message: edited pcb
Parts:
- Q1, Q2: value Q_NPN_BEC -> MMBT8050LT1G_BEC
- U2: value MCP16311-MNY -> AMS1117-5
- U6: value BD00GA5WEFJ -> AMS1117-3.3
Connections:
- L1 pad 1: Net-(C9-Pad2) -> Net-(L1-Pad1)
- U2 pad 2: Net-(C7-Pad1) -> Net-(L1-Pad1)
- U2 pad 4: Vin -> (no net)
- U2 pad 5: GND -> (no net)
- U2 pad 6: Net-(C9-Pad2) -> (no net)
- U2 pad 7: Net-(C9-Pad1) -> (no net)
- U2 pad 8: GND -> (no net)
- U6 pad 1: +3V3 -> Net-(R20-Pad2)
- U6 pad 2: Net-(R20-Pad2) -> +3V3
- U6 pad 3: GND -> +5V
- U6 pad 4: Net-(U6-Pad4) -> (no net)
- U6 pad 5: +5V -> (no net)
- U6 pad 6: Net-(U6-Pad6) -> (no net)
- U6 pad 7: Net-(U6-Pad7) -> (no net)
- U6 pad 8: +5V -> (no net)
- U6 pad 9: GND -> (no net)
Other:
- net class Default: trace_width 0.4 -> 0.25

Commit message: pcb layout hoan chỉnh
Parts:
- removed C7: 1uF, ESP8266:C_0603
- removed C9: 100nF, ESP8266:C_0603
- removed G***: LOGO, ESP8266:RST
- removed G***: LOGO, ESP8266:logo_cc-bby-sa_14.1x5mm
- removed G***: LOGO, ESP8266:GPIO0
- removed G***: LOGO, ESP8266:logo-iotmakervn_7
- removed G***: LOGO, ESP8266:logo-jack-5528
- removed G***: LOGO, ESP8266:logo-jack_7.4x3
- removed G***: LOGO, ESP8266:LEDPWR
- removed G***: LOGO, ESP8266:GPIO16
- removed G***: LOGO, ESP8266:logo-iotmakervn_7.5x5
- removed G***: LOGO, ESP8266:logo_openhardware_5x5mm
- P1, P2: footprint Pin_Headers:Pin_Header_Straight_1x08 -> Pin_Headers:Pin_Header_Straight_1x08_Pitch1.27mm
- P3: footprint Pin_Headers:Pin_Header_Straight_1x06 -> Pin_Headers:Pin_Header_Straight_1x06_Pitch1.27mm
- P4: footprint Pin_Headers:Pin_Header_Straight_1x10 -> Pin_Headers:Pin_Header_Straight_1x10_Pitch1.27mm
- P5: footprint Pin_Headers:Pin_Header_Straight_1x04 -> Pin_Headers:Pin_Header_Straight_1x04_Pitch1.27mm
- U2: footprint Housings_SSOP:MSOP-8_3x3mm_Pitch0.65mm -> TO_SOT_Packages_SMD:SOT-223
- U6: footprint ESP8266:HTSOP-J8 -> TO_SOT_Packages_SMD:SOT-223
- moved C12 117.4 mm to (247.3, 98.9), turned to 90 degrees
- moved P4 112.5 mm to (238.7, 82.3)
- moved C3 108.2 mm to (233.2, 105.6), turned to 0 degrees
- moved P2 108.0 mm to (243.3, 129.6)
- moved CON1 106.6 mm to (221.5, 121.5)
- moved R6 106.6 mm to (233.2, 100.9), turned to 90 degrees
- moved R7 106.2 mm to (234.9, 100.8), turned to 90 degrees
- moved C6 106.2 mm to (230.8, 100.9), turned to 270 degrees
- moved C2 105.9 mm to (228.5, 100.9), turned to 270 degrees
- moved X1 105.2 mm to (224.7, 101.0), turned to 0 degrees
- moved C4 105.2 mm to (226.0, 105.7), turned to 180 degrees
- moved Q2 105.2 mm to (239.0, 96.9), turned to 180 degrees
- moved R10 104.9 mm to (238.6, 100.9), turned to 180 degrees
- moved Q1 104.9 mm to (238.8, 106.1), turned to 180 degrees
- moved R11 104.9 mm to (238.6, 103.1), turned to 180 degrees
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Routing:
- net MOSI: track 38.5 -> 109.8 mm, vias 2 -> 10
- net Vin: track 55.8 -> 119.5 mm, vias 3 -> 5
- net GND: track 311.7 -> 266.5 mm, vias 15 -> 7
- net REST: track 114.1 -> 72.9 mm, vias 1 -> 5
- net XO: track 10.6 -> 45.9 mm, vias 0 -> 2
- net SCLK: track 38.9 -> 73.6 mm, vias 2 -> 4
- net GPIO10: track 37.7 -> 70.7 mm, vias 2 -> 5
- net GPIO4: track 133.8 -> 165.1 mm, vias 3 -> 1
- net GPIO5: track 128.7 -> 159.1 mm, vias 4 -> 1
- net GPIO15: track 47.2 -> 77.3 mm, vias 2 -> 4
- net Net-(R7-Pad2): track 4.11 -> 30.4 mm, vias 0 -> 2
- net GPIO2: track 44.0 -> 70.2 mm, vias 2 -> 3
- net TXD: track 82.6 -> 108.5 mm, vias 1 -> 7
- net Net-(C9-Pad2): track 25.6 -> 0.00 mm
- net RXD: track 81.0 -> 106.2 mm, vias 2 -> 5
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Other:
- board outline removed
- net class Default: clearance 0.254 -> 0.2; trace_width 0.25 -> 0.4; via_dia 1.1 -> 0.8; via_drill 0.6 -> 0.4
- net class Power added: clearance 0.2, trace_width 0.8, via_dia 0.8, via_drill 0.4
- rule trace_clearance: 0.254 -> 0.2
- rule trace_min: 0.254 -> 0.2
- board text removed: "3.3V"
- board text removed: "5V"
- board text removed: "ADC"
- board text removed: "CSO"
- board text removed: "GND"
- board text removed: "GPIO0"
- board text removed: "GPIO02"
- board text removed: "GPIO04"
- board text removed: "GPIO05"
- board text removed: "GPIO09"
- board text removed: "GPIO10"
- board text removed: "GPIO12"
- board text removed: "GPIO13"
- board text removed: "GPIO14"
- board text removed: "GPIO15"
- board text removed: "GPIO16"
- board text removed: "MISO"
- board text removed: "MOSI"
- board text removed: "RST"
- board text removed: "RXD"
- board text removed: "SCL/GPIO5"
- board text removed: "SCLK"
- board text removed: "SDA/GPIO4"
- board text removed: "TXD"
- board text removed: "VIN"
- board text removed: "https://esp8266.vn"

Commit message: pcb hoàn chỉnh, add 3d, khung
Other:
- board outline added: 64 x 52.8 mm
- net class Default: trace_width 0.4 -> 0.25
Changed lines of the file:
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@@
   (general
     (thickness 1.6)
-    (drawings 35)
+    (drawings 61)
     (tracks 1506)
     (zones 0)
@@
   )
   (setup
-    (last_trace_width 0.4)
+    (last_trace_width 0.25)
     (trace_clearance 0.2)
     (zone_clearance 0.508)
@@
   (net_class Default "This is the default net class."
     (clearance 0.2)
-    (trace_width 0.4)
+    (trace_width 0.25)
     (via_dia 0.8)
     (via_drill 0.4)
@@
       (rotate (xyz 0 0 0))
     )
+    (model ${KIPRJMOD}/lib/ESP8266.3dshapes/C_0603.wrl
+      (at (xyz 0 0 0))
+      (scale (xyz 1 1 1))
+      (rotate (xyz 0 0 0))
+    )
   )
   (module ESP8266:C_0603 (layer F.Cu)
@@
       (net 1 GND))
     (model Capacitors_SMD.3dshapes/C_0603_HandSoldering.wrl
+      (at (xyz 0 0 0))
+      (scale (xyz 1 1 1))
+      (rotate (xyz 0 0 0))
+    )
+    (model ${KIPRJMOD}/lib/ESP8266.3dshapes/C_0603.wrl
       (at (xyz 0 0 0))
       (scale (xyz 1 1 1))
@@
       (net 4 Vin))
     (model Capacitors_SMD.3dshapes/C_1210_HandSoldering.wrl
+      (at (xyz 0 0 0))
+      (scale (xyz 1 1 1))
+      (rotate (xyz 0 0 0))
+    )
+    (model ${KIPRJMOD}/lib/ESP8266.3dshapes/C_1210.wrl
       (at (xyz 0 0 0))
       (scale (xyz 1 1 1))
@@
       (rotate (xyz 0 0 0))
     )
+    (model ${KIPRJMOD}/lib/ESP8266.3dshapes/C_1210.wrl
+      (at (xyz 0 0 0))
+      (scale (xyz 1 1 1))
+      (rotate (xyz 0 0 0))
+    )
   )
   (module ESP8266:C_0603 (layer F.Cu)
@@
       (net 5 REST))
     (model Capacitors_SMD.3dshapes/C_0603_HandSoldering.wrl
+      (at (xyz 0 0 0))
+      (scale (xyz 1 1 1))
+      (rotate (xyz 0 0 0))
+    )
+    (model ${KIPRJMOD}/lib/ESP8266.3dshapes/C_0603.wrl
       (at (xyz 0 0 0))
       (scale (xyz 1 1 1))
@@
       (rotate (xyz 0 0 0))
     )
+    (model ${KIPRJMOD}/lib/ESP8266.3dshapes/C_0603.wrl
+      (at (xyz 0 0 0))
+      (scale (xyz 1 1 1))
+      (rotate (xyz 0 0 0))
+    )
   )
   (module ESP8266:C_0603 (layer F.Cu)
@@
       (net 1 GND))
     (model Capacitors_SMD.3dshapes/C_0603_HandSoldering.wrl
+      (at (xyz 0 0 0))
+      (scale (xyz 1 1 1))
+      (rotate (xyz 0 0 0))
+    )
+    (model ${KIPRJMOD}/lib/ESP8266.3dshapes/C_0603.wrl
       (at (xyz 0 0 0))
       (scale (xyz 1 1 1))
@@
       (rotate (xyz 0 0 0))
     )
+    (model ${KIPRJMOD}/lib/ESP8266.3dshapes/C_1210.wrl
+      (at (xyz 0 0 0))
+      (scale (xyz 1 1 1))
+      (rotate (xyz 0 0 0))
+    )
   )
   (module ESP8266:C_1210 (layer F.Cu)
@@
       (rotate (xyz 0 0 0))
     )
+    (model ${KIPRJMOD}/lib/ESP8266.3dshapes/C_1210.wrl
+      (at (xyz 0 0 0))
+      (scale (xyz 1 1 1))
+      (rotate (xyz 0 0 0))
+    )
   )
   (module ESP8266:C_0603 (layer F.Cu)
@@
       (net 6 +3V3))
     (model Capacitors_SMD.3dshapes/C_0603_HandSoldering.wrl
+      (at (xyz 0 0 0))
+      (scale (xyz 1 1 1))
+      (rotate (xyz 0 0 0))
+    )
+    (model ${KIPRJMOD}/lib/ESP8266.3dshapes/C_0603.wrl
       (at (xyz 0 0 0))
       (scale (xyz 1 1 1))
@@
       (rotate (xyz 0 0 0))
     )
+    (model ${KIPRJMOD}/lib/ESP8266.3dshapes/C_1210.wrl
+      (at (xyz 0 0 0))
+      (scale (xyz 1 1 1))
+      (rotate (xyz 0 0 0))
+    )
   )
   (module ESP8266:C_0603 (layer F.Cu)
@@
       (rotate (xyz 0 0 0))
     )
+    (model ${KIPRJMOD}/lib/ESP8266.3dshapes/C_0603.wrl
+      (at (xyz 0 0 0))
+      (scale (xyz 1 1 1))
+      (rotate (xyz 0 0 0))
+    )
   )
   (module ESP8266:C_0603 (layer F.Cu)
@@
       (net 6 +3V3))
     (model Capacitors_SMD.3dshapes/C_0603_HandSoldering.wrl
+      (at (xyz 0 0 0))
+      (scale (xyz 1 1 1))
+      (rotate (xyz 0 0 0))
+    )
+    (model ${KIPRJMOD}/lib/ESP8266.3dshapes/C_0603.wrl
       (at (xyz 0 0 0))
       (scale (xyz 1 1 1))
@@
     (pad 1 thru_hole rect (at 0 0) (size 3.5 3.5) (drill oval 1 3) (layers *.Cu *.Mask)
       (net 8 "Net-(CON1-Pad1)"))
+    (model ${KIPRJMOD}/lib/ESP8266.3dshapes/dc_socket.wrl
+      (at (xyz -0.2362204724409449 0 0))
+      (scale (xyz 1 1 1))
+      (rotate (xyz 180 180 -90))
+    )
   )
   (module ESP8266:do214aa-g (layer F.Cu)
@@
       (rotate (xyz 0 0 180))
     )
+    (model ${KIPRJMOD}/lib/ESP8266.3dshapes/do214aa.wrl
+      (at (xyz 0 0 0))
+      (scale (xyz 1 1 1))
+      (rotate (xyz 0 0 0))
+    )
   )
   (module Choke_SMD:Choke_SMD_Wuerth-WE-PD2-Typ-MS (layer F.Cu)
@@
     (pad 1 smd rect (at -1.9304 0) (size 2.14884 5.4991) (layers F.Cu F.Paste F.Mask)
       (net 14 "Net-(L1-Pad1)"))
+    (model ${KIPRJMOD}/lib/ESP8266.3dshapes/inductor_smd_8x5mm.wrl
+      (at (xyz 0 0 0))
+      (scale (xyz 1 1 1))
+      (rotate (xyz 0 0 0))
+    )
   )
   (module Pin_Headers:Pin_Header_Straight_1x08_Pitch1.27mm (layer F.Cu)
@@
     (pad 1 smd rect (at -1.3 -1.35) (size 1.35 0.4) (layers F.Cu F.Paste F.Mask)
       (net 11 VCC))
+    (model ${KIPRJMOD}/lib/ESP8266.3dshapes/AB2_USB_MICRO_SMD.wrl
+      (at (xyz 0 -0.5118110236220472 0))
+      (scale (xyz 0.5 1 0.4001))
+      (rotate (xyz 0 0 0))
+    )
   )
   (module ESP8266:ESP-12F (layer F.Cu)
@@
     (pad 22 smd roundrect (at 14 0 270) (size 2.5 1.1) (drill (offset 0.7 0)) (layers F.Cu F.Paste F.Mask)(roundrect_rratio 0.25)
       (net 16 TXD))
-    (model ${ESPLIB}/ESP8266.3dshapes/ESP-12.wrl
-      (at (xyz 0.04 0 0))
-      (scale (xyz 0.3937 0.3937 0.3937))
+    (model ${KIPRJMOD}/lib/ESP8266.3dshapes/ESP-12.wrl
+      (at (xyz 0.05905511811023623 -0.09842519685039371 -0.01968503937007874))
+      (scale (xyz 0.3 0.3001 0.2))
       (rotate (xyz 0 0 0))
     )
@@
     (model Crystals.3dshapes/Crystal_SMD_5032_4Pads.wrl
       (at (xyz 0 0 0))
-      (scale (xyz 0.6 1 1))
-      (rotate (xyz 0 0 0))
-    )
-  )
+      (scale (xyz 0.0001 0.0001 1))
+      (rotate (xyz 0 0 0))
+    )
+    (model ${KIPRJMOD}/lib/ESP8266.3dshapes/Crystal_SMD_5032-2pin_5.0x3.2mm.wrl
+      (at (xyz 0 0 0))
+      (scale (xyz 0.4 0.6 1))
+      (rotate (xyz 0 0 0))
+    )
+  )
+  (gr_line (start 206.629 78.994) (end 206.9465 79.0575) (angle 90) (layer Edge.Cuts) (width 0.15))
+  (gr_line (start 206.629 82.1055) (end 206.629 78.994) (angle 90) (layer Edge.Cuts) (width 0.15))
+  (gr_line (start 206.629 93.9165) (end 206.629 82.1055) (angle 90) (layer Edge.Cuts) (width 0.15))
+  (gr_line (start 206.629 105.156) (end 206.629 93.9165) (angle 90) (layer Edge.Cuts) (width 0.15))
+  (gr_line (start 206.629 111.76) (end 206.629 105.156) (angle 90) (layer Edge.Cuts) (width 0.15))
+  (gr_line (start 206.629 131.7625) (end 206.629 111.76) (angle 90) (layer Edge.Cuts) (width 0.15))
+  (gr_line (start 216.3445 131.7625) (end 206.629 131.7625) (angle 90) (layer Edge.Cuts) (width 0.15))
+  (gr_line (start 226.06 131.7625) (end 216.3445 131.7625) (angle 90) (layer Edge.Cuts) (width 0.15))
+  (gr_line (start 243.078 131.7625) (end 226.06 131.7625) (angle 90) (layer Edge.Cuts) (width 0.15))
+  (gr_line (start 252.6665 131.7625) (end 243.078 131.7625) (angle 90) (layer Edge.Cuts) (width 0.15))
+  (gr_line (start 267.589 131.6355) (end 252.6665 131.7625) (angle 90) (layer Edge.Cuts) (width 0.15))
+  (gr_line (start 270.637 129.0955) (end 267.589 131.6355) (angle 90) (layer Edge.Cuts) (width 0.15))
+  (gr_line (start 270.637 121.7295) (end 270.637 129.0955) (angle 90) (layer Edge.Cuts) (width 0.15))
+  (gr_line (start 270.637 117.729) (end 270.637 121.7295) (angle 90) (layer Edge.Cuts) (width 0.15))
+  (gr_line (start 270.637 112.0775) (end 270.637 117.729) (angle 90) (layer Edge.Cuts) (width 0.15))
+  (gr_line (start 270.637 105.6005) (end 270.637 112.0775) (angle 90) (layer Edge.Cuts) (width 0.15))
+  (gr_line (start 270.637 99.949) (end 270.637 105.6005) (angle 90) (layer Edge.Cuts) (width 0.15))
+  (gr_line (start 267.716 96.4565) (end 270.637 99.949) (angle 90) (layer Edge.Cuts) (width 0.15))
+  (gr_line (start 267.716 92.456) (end 267.716 96.4565) (angle 90) (layer Edge.Cuts) (width 0.15))
+  (gr_line (start 267.716 84.8995) (end 267.716 92.456) (angle 90) (layer Edge.Cuts) (width 0.15))
+  (gr_line (start 261.366 79.0575) (end 267.716 84.8995) (angle 90) (layer Edge.Cuts) (width 0.15))
+  (gr_line (start 253.238 79.0575) (end 261.366 79.0575) (angle 90) (layer Edge.Cuts) (width 0.15))
+  (gr_line (start 236.982 79.0575) (end 253.238 79.0575) (angle 90) (layer Edge.Cuts) (width 0.15))
+  (gr_line (start 223.393 79.0575) (end 236.982 79.0575) (angle 90) (layer Edge.Cuts) (width 0.15))
+  (gr_line (start 215.138 79.0575) (end 223.393 79.0575) (angle 90) (layer Edge.Cuts) (width 0.15))
+  (gr_line (start 206.756 79.121) (end 215.138 79.0575) (angle 90) (layer Edge.Cuts) (width 0.15))
   (gr_circle (center 218.567 80.7085) (end 217.6145 79.756) (layer Eco2.User) (width 0.2))
   (gr_line (start 206.756 80.4545) (end 206.756 78.9305) (angle 90) (layer Eco2.User) (width 0.2))
